File: boards/bluetooth/layout/bluetooth.kicad_sch (KiCad schematic)
At the start: 9 parts, among them U1 HM-19

Commit message: 🐛 Identify the Bluetooth module on CC and pull its RESETB up
M6: the plug's CC1 and CC2 join its D+ contacts. The main board's UART4 TX
idles high and pulls its CC contacts (5.1 kOhm Rd each) to about 3.2 V
through them, a level no USB Type-C source makes across a sink's Rd (R2.0
Tables 4-35, 4-36: 2.18 / 2.04 V max), so the main board can switch 3V3
onto SBU only for the module and leave SBU open for every USB partner.

m17: R4 10 kOhm from HM-19 RESETB to 3V3; the CC2640R2F's RESET_N has no
internal pull-up (SWRS204C Table 7-1).

The board's minimum silkscreen text height is 0.5 mm, the size of its
reference designators. The layout gets the packages' new courtyards and R4,
not yet placed.
Parts:
- added R4: 10k 1% 100mW, stdlib_kicad-footprints_Resistor_SMD:R_0603_1608Metric, symbol R_Small
Connections:
- net 3V3: now also R4.2
- net UART_RX: now also USB1.11 (CC2), USB1.3 (CC1)
- net RESETB: now reaches U1.11 (RESETB)
- net RESETB: now also R4.1
- no-connect marks 15 -> 13
Changed lines of the file:
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@@
-	)
-	(no_connect
-		(at 129.54 59.69)
 	)
 	(no_connect
@@
 	)
 	(no_connect
-		(at 129.54 62.23)
-	)
-	(no_connect
 		(at 129.54 54.61)
 	)
@@
 	(wire
 		(pts
+			(xy 208.28 88.9) (xy 208.28 83.82)
+		)
+		(stroke
+			(width 0)
+			(type default)
+		)
+	)
+	(wire
+		(pts
 			(xy 129.54 90.17) (xy 119.38 90.17)
 		)
@@
 			(width 0)
 			(type default)
+		)
+	)
+	(label "UART_RX"
+		(at 129.54 62.23 180)
+		(effects
+			(font
+				(size 1.27 1.27)
+			)
+			(justify right bottom)
+		)
+	)
+	(label "UART_RX"
+		(at 129.54 59.69 180)
+		(effects
+			(font
+				(size 1.27 1.27)
+			)
+			(justify right bottom)
+		)
+	)
+	(label "RESETB"
+		(at 73.66 67.31 180)
+		(effects
+			(font
+				(size 1.27 1.27)
+			)
+			(justify right bottom)
 		)
 	)
@@
 			)
 			(justify left bottom)
+		)
+	)
+	(label "RESETB"
+		(at 208.28 93.98 270)
+		(effects
+			(font
+				(size 1.27 1.27)
+			)
+			(justify right bottom)
 		)
 	)
@@
 					(unit 1)
 				)
+			)
+		)
+	)
+	(symbol
+		(lib_id "VCC")
+		(at 208.28 83.82 0)
+		(unit 1)
+		(body_style 1)
+		(exclude_from_sim no)
+		(in_bom yes)
+		(on_board yes)
+		(in_pos_files yes)
+		(dnp no)
+		(fields_autoplaced yes)
+		(property "Reference" "#PWR2636336ce09a5417b1794783b9b978de"
+			(at 208.28 83.82 0)
+			(hide yes)
+			(show_name no)
+			(do_not_autoplace no)
+			(effects
+				(font
+					(size 1.27 1.27)
+				)
+			)
+		)
+		(property "Value" "3V3"
+			(at 208.28 80.01 0)
+			(show_name no)
+			(do_not_autoplace no)
+			(effects
+				(font
+					(size 1.27 1.27)
+				)
+			)
+		)
+		(property "Footprint" ""
+			(at 208.28 83.82 0)
+			(hide yes)
+			(show_name no)
+			(do_not_autoplace no)
+			(effects
+				(font
+					(size 1.27 1.27)
+				)
+			)
+		)
+		(property "Datasheet" ""
+			(at 208.28 83.82 0)
+			(hide yes)
+			(show_name no)
+			(do_not_autoplace no)
+			(effects
+				(font
+					(size 1.27 1.27)
+				)
+			)
+		)
+		(property "Description" "Power symbol creates a global label with name \"VCC\""
+			(at 208.28 83.82 0)
+			(hide yes)
+			(show_name no)
+			(do_not_autoplace no)
+			(effects
+				(font
+					(size 1.27 1.27)
+				)
+			)
+		)
+		(property "ki_keywords" "global power"
+			(at 208.28 83.82 0)
+			(hide yes)
+			(show_name no)
+			(do_not_autoplace no)
+			(effects
+				(font
+					(size 1.27 1.27)
+				)
+			)
+		)
+		(pin "1"
+		)
+		(instances
+			(project "bluetooth"
+				(path "/513d9cc1-d27a-514d-a37c-2f1ca04dddfa"
+					(reference "#PWR2636336ce09a5417b1794783b9b978de")
+					(unit 1)
+				)
+			)
+		)
+	)
+	(symbol
+		(lib_id "R_Small")
+		(at 208.28 91.44 180)
+		(unit 1)
+		(body_style 1)
+		(exclude_from_sim no)
+		(in_bom yes)
+		(on_board yes)
+		(in_pos_files yes)
+		(dnp no)
+		(fields_autoplaced yes)
+		(property "Reference" "R4"
+			(at 210.82 90.805 0)
+			(show_name no)
+			(do_not_autoplace no)
+			(effects
+				(font
+					(size 1.016 1.016)
+				)
+				(justify right)
+			)
+		)
+		(property "Value" "10k 1% 100mW"
+			(at 210.82 92.075 0)
+			(show_name no)
+			(do_not_autoplace no)
+			(effects
+				(font
+					(size 1.27 1.27)
+				)
+				(justify right)
+			)
+		)
+		(property "Footprint" "stdlib_kicad-footprints_Resistor_SMD:R_0603_1608Metric"
+			(at 208.28 91.44 0)
+			(hide yes)
+			(show_name no)
+			(do_not_autoplace no)
+			(effects
+				(font
+					(size 1.27 1.27)
+				)
+			)
+		)
+		(property "Datasheet" ""
+			(at 208.28 91.44 0)
+			(hide yes)
+			(show_name no)
+			(do_not_autoplace no)
+			(effects
+				(font
+					(size 1.27 1.27)
+				)
+			)
+		)
+		(property "Description" "10k 1% 100mW"
+			(at 208.28 91.44 0)
+			(hide yes)
+			(show_name no)
+			(do_not_autoplace no)
+			(effects
+				(font
+					(size 1.27 1.27)
+				)
+			)
+		)
+		(property "Path" "R4.R"
+			(at 208.28 91.44 0)
+			(hide yes)
+			(show_name no)
+			(do_not_autoplace no)
+			(effects
+				(font
+					(size 1.27 1.27)
+				)
+			)
+		)
+		(pin "1"
+		)
+		(pin "2"
+		)
+		(instances
+			(project "bluetooth"
+				(path "/513d9cc1-d27a-514d-a37c-2f1ca04dddfa"
+					(reference "R4")
+					(unit 1)
+				)
