File: boards/main/layout/main.kicad_pcb (KiCad board)
At the start: 4 copper layers, 50 x 90 mm, 193 parts, among them IC1 STM32H725RGV6, IC2 LSM6DSVTR, IC3 TSC2020IYST, IC4 TSC2020IYST, IC5 L6205D013TR, IC6 STSPIN958TR, IC7 L6981C33DR, J1 B02B-PASK(LF)(SN), M1 B02B-PASK(LF)(SN), M2 B02B-PASK(LF)(SN), M3 B02B-PASK(LF)(SN), P1 SM05B-SRSS-TB(LF)(SN), Q1 AO3400A, Q2 AO3400A, Q3 AO3400A, Q4 AO3400A, Q5 AO3400A, Q6 HSBB3072, Q7 AO3401A, SW1 DSHP04TJGER, SW2 GT-TC048B-H025-L1, SW3 GT-TC048B-H025-L1, SW4 MK-12D18-G040, SW5 GT-TC048B-H025-L1, U1 TPS61178RNWR, U2 GT-USB-7010ASV, U4 TPS2121RUXR, U5 LM66100DCKR, U6 USBLC6-2SC6, U7 TLV7041DBVR

Commit message: ♻️ Give the main layout main's pour settings and clear what the 2512 shunts touch
boards/main/layout/finish.py, one-off after usb_wall.py: the teardrop, pour, inner-plane relief,
screw-hole void, mask and LED settings that previous/transfer_layout.py gives a fresh transfer
(the earlier scripts name copper with random UUIDs, so they do not replay on a new transfer);
C33 above C32, clear of R31's 2512 courtyard; the SBU_DET_A via off R33's pad; C69/C70's 3V3
from EC1 pin 5, their vias being in H2's plane void; three bumps on D- that match the USB pair;
and the teardrops a 0.1 mm fill leaves alone or that make copper slivers (found by removing each
and re-running DRC).
Parts:
- moved C33 1.87 mm to (143.6, 121.6), turned to 180 degrees
Routing:
- net USBD_N: track 117.4 -> 121.7 mm
- net DRIVERS.FAN_VSPUMP: track 2.61 -> 5.13 mm
- net 3V3: track 125.6 -> 126.5 mm, vias 47 -> 45
- net DRIVERS.FAN_VBOOT: track 2.57 -> 1.86 mm
- removed copper zone on B.Cu, net Current_Sensor_Left
- removed copper zone on F.Cu, net Current_Sensor_Left
- removed copper zone on B.Cu, net Current_Sensor_Right
- removed copper zone on F.Cu, net Current_Sensor_Right
- removed copper zone on F.Cu, net Motor_L_Sense+
- removed copper zone on B.Cu, net Motor_L_Sense-
- removed copper zone on F.Cu, net Motor_L_Sense-
- removed copper zone on F.Cu, net Motor_R_Sense+
- removed copper zone on F.Cu, net Motor_R_Sense-
- removed copper zone on B.Cu, net PERIPHERALS.USB_CC2
- removed copper zone on B.Cu, net REGULATORS.BAT_SW_GATE
- removed copper zone on F.Cu, net SENSORS.WALL0_LED_A
- removed copper zone on B.Cu, net VBAT
- removed copper zone on F.Cu, net Wall_Sensor_PWM_3
Other:
- rule pad_to_mask_clearance: 0 -> 0.02
