File: boards/main/layout/main.kicad_sch (KiCad schematic)
At the start: 193 parts, among them IC1 STM32H725RGV6, IC2 LSM6DSVTR, IC3 TSC2020IYST, IC4 TSC2020IYST, IC5 L6205D013TR, IC6 STSPIN958TR, IC7 L6981C33DR, J1 B02B-PASK(LF)(SN), M1 B02B-PASK(LF)(SN), M2 B02B-PASK(LF)(SN), M3 B02B-PASK(LF)(SN), P1 SM05B-SRSS-TB(LF)(SN), Q1 AO3400A, Q2 AO3400A, Q3 AO3400A, Q4 AO3400A, Q5 AO3400A, Q6 HSBB3072, Q7 AO3401A, SW1 DSHP04TJGER, SW2 GT-TC048B-H025-L1, SW3 GT-TC048B-H025-L1, SW4 MK-12D18-G040, SW5 GT-TC048B-H025-L1, U1 TPS61178RNWR, U2 GT-USB-7010ASV, U4 TPS2121RUXR, U5 LM66100DCKR, U6 USBLC6-2SC6, U7 TLV7041DBVR

Commit message: ✨ Bypass U6's rail pin with C79 and set the designators to 0.5 mm / 0.125 mm
USBLC6-2 DocID 11265 Figure 18 puts CBUS = 100 nF on the VBUS pin: C79
(0402 X7R, CL05B104KB54PNC, basic) on 3V3 above U6, placed and routed by
boards/main/layout/rail_silk.py, declared under M12.

The owner chose 0.5 mm high, 0.125 mm stroke silkscreen designators (KiCad's
stroke clamp at 0.5 mm): rail_silk.py resizes every designator and P1's
labels and re-places the two whose spot changed; the board minimum stroke is
0.125 mm.
Parts:
- added C79: 100nF 10% 50V X7R, stdlib_kicad-footprints_Capacitor_SMD:C_0402_1005Metric, symbol C_Small
Connections:
- net 3V3: now also C79.2
- net GND: now also C79.1
Other:
- moved on the sheet: C18, C19, C24, C25, C26, C27, C28, C29, C3, C34, C35, C36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

Commit message: 🔧 Use the top-entry JST BM05B-SRSS-TB for the SWD connector P1
The previous revision had an upright 2.54 mm header at this spot, so an upright plug fits the chassis; the side-entry SM05B-SRSS-TB was never needed. New package components/jst/BM05B-SRSS-TB (KiCad library footprint checked against the JST SH catalogue's top-entry land pattern, STEP embedded, test bench), LCSC C160391; the SM05B-SRSS-TB package goes. swd_top.py places P1 where the side-entry header was, contacts inwards, and routes its five nets at 45 degrees.
Parts:
- P1: value SM05B-SRSS-TB(LF)(SN) -> BM05B-SRSS-TB(LF)(SN); footprint Team-Micras_MicrasPCB_components_jst_SM05B-SRSS-TB:JST_SH_SM05B-SRSS-TB_1x05-1MP_P1.00mm_Horizontal -> Team-Micras_MicrasPCB_components_jst_BM05B-SRSS-TB:JST_SH_BM05B-SRSS-TB_1x05-1MP_P1.00mm_Vertical; symbol SM05B-SRSS-TB -> BM05B-SRSS-TB
Changed lines of the file:
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@@
 	)
 	(symbol
-		(lib_id "SM05B-SRSS-TB")
+		(lib_id "BM05B-SRSS-TB")
 		(at 1283.97 252.73 0)
 		(unit 1)
@@
 			)
 		)
-		(property "Value" "SM05B-SRSS-TB(LF)(SN)"
+		(property "Value" "BM05B-SRSS-TB(LF)(SN)"
 			(at 1290.32 253.365 0)
 			(show_name no)
@@
 			)
 		)
-		(property "Footprint" "Team-Micras_MicrasPCB_components_jst_SM05B-SRSS-TB:JST_SH_SM05B-SRSS-TB_1x05-1MP_P1.00mm_Horizontal"
+		(property "Footprint" "Team-Micras_MicrasPCB_components_jst_BM05B-SRSS-TB:JST_SH_BM05B-SRSS-TB_1x05-1MP_P1.00mm_Vertical"
 			(at 1283.97 252.73 0)
 			(hide yes)
@@
 			)
 		)
-		(property "Description" "JST SH header 1x05, 1.00 mm pitch, side entry, SMD, two reinforcement pads (JST SM05B-SRSS-TB)"
+		(property "Description" "JST SH header 1x05, 1.00 mm pitch, top entry, SMD, two reinforcement pads (JST BM05B-SRSS-TB)"
 			(at 1283.97 252.73 0)
 			(hide yes)
