File: boards/main/layout/REGULATORS.kicad_sch (KiCad schematic)
At the start: 41 parts, among them IC7 L6981C33DR, J1 B02B-PASK(LF)(SN), Q6 HSBB3072, SW4 MK-12D18-G040, U1 TPS61178RNWR, U4 TPS2121RUXR, U5 LM66100DCKR

Commit message: 🏷️ Name the main board's module ports after their nets
A sheet pin and its hierarchical label take the module's port name and the root's label the net
name; KiCad's ERC flagged the 33 nets whose two names differed only in case (similar_labels).
GND_BAT becomes a ground port of REGULATORS, so the root shows a power symbol at its sheet pin
instead of a label nothing else joined (label_dangling).
Other:
- moved on the sheet: C42, C43, C44, C45, C46, C47, C48, C49, C50, C51, C52, C53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

Commit message: 🎨 Place the main board's REGULATORS sheet
Other:
- note added: "20 V boost: TPS61178 for the L6205 bridges, on while Motors_Enable is high"
- note added: "3V3 buck: L6981C33 from VSYS"
- note added: "Battery input and switch: J1, SW4, low-side Q6"
- note added: "Battery measurement: to PA5"
- note added: "SWD probe supply: LM66100 ideal diode"
- note added: "Sheet ports"
- note added: "Supply selection: TPS2121, the higher of VBAT and +5V on VSYS"
- title: (none) -> Battery, supply selection and regulators
- moved on the sheet: C42, C43, C44, C45, C46, C47, C48, C49, C50, C51, C52, C53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
