File: boards/main/layout/DRIVERS.kicad_sch (KiCad schematic)
At the start: 31 parts, among them IC5 L6205D013TR, IC6 STSPIN958TR, M1 B02B-PASK(LF)(SN), M2 B02B-PASK(LF)(SN), M3 B02B-PASK(LF)(SN)

Commit message: ✨ Place the schematics from per-sheet placement files: the tool's fixes, the B02B pin names, docs, and the encoder, Bluetooth and DRIVERS placements for this revision
Parts:
- removed C65, C66: 10uF 10% 50V X5R, stdlib_kicad-footprints_Capacitor_SMD:C_0805_2012Metric, symbol C_Small
- removed R49: 100k 1%, stdlib_kicad-footprints_Resistor_SMD:R_0402_1005Metric, symbol R_Small
Connections:
- net 3V3: now also IC6.12 (PWM2/PH)
- net GND: no longer IC6.12 (PWM2/PH)
- net Motor_L_Sense+: now also IC5.7 (OUT1B), R33.2; no longer IC5.4 (OUT1A), R32.2
- net Motor_L_Sense-: now also M2.2 (Pin_2), R33.1; no longer M1.2 (Pin_2), R32.1
- net Motor_R_Sense+: now also IC5.4 (OUT1A), R32.2; no longer IC5.7 (OUT1B), R33.2
- net Motor_R_Sense-: now also M1.2 (Pin_2), R32.1; no longer M2.2 (Pin_2), R33.1
- net Fan_TOFF renamed Fan_Overcurrent
- net Motors_Enable renamed Motor_Enable
Other:
- note removed: "Fan driver: STSPIN958, current limit through R31"
- note removed: "Motor bridge: L6205, current sense through R32 and R33"
- note removed: "Sheet ports"
- title: Motor and fan drivers -> (none)
- moved on the sheet: C30, C31, C32, C33, C34, C35, C36, C37, C38, C39, C40, C41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

Commit message: 🎨 Place this revision's root, REGULATORS and SENSORS sheets; give the CJA1117B room for its pin names
Other:
- note added: "Fan driver: STSPIN958, current limit through R31"
- note added: "Motor bridge: L6205, current sense through R32 and R33"
- note added: "Sheet ports"
- title: (none) -> Motor and fan drivers
- moved on the sheet: C30, C31, C32, C33, C34, C35, C36, C37, C38, C39, C40, C41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
