File: boards/main/layout/SENSORS.kicad_sch (KiCad schematic)
At the start: 35 parts, among them IC2 LSM6DSVTR, IC3 TSC2020IYST, IC4 TSC2020IYST, Q2 AO3400A, Q3 AO3400A, Q4 AO3400A, Q5 AO3400A

Commit message: 🎨 Place this revision's root, REGULATORS and SENSORS sheets; give the CJA1117B room for its pin names
Other:
- note added: "Encoder slots: EC1 right wheel, EC2 left wheel"
- note added: "IMU: LSM6DSV on the shared SPI bus"
- note added: "Motor current: TSC2020, 20 V/V across the 40 mOhm shunts"
- note added: "Sheet ports"
- note added: "Wall sensor 0: W1, emitter switch Q2"
- note added: "Wall sensor 1: W2, emitter switch Q3"
- note added: "Wall sensor 2: W3, emitter switch Q4"
- note added: "Wall sensor 3: W4, emitter switch Q5"
- title: (none) -> IMU, current sensors, wall sensors and encoder slots
- moved on the sheet: C24, C25, C26, C27, C28, C29, EC1, EC2, IC2, IC3, IC4, Q2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
