File: boards/main/layout/SENSORS.kicad_sch (KiCad schematic)
At the start: 49 parts, among them IC2 LSM6DSVTR, IC3 TSC2020IYST, IC4 TSC2020IYST, Q2 AO3400A, Q3 AO3400A, Q4 AO3400A, Q5 AO3400A

Commit message: 🎨 Place the main board's SENSORS sheet, and size the ports column for global labels' flags
Other:
- note added: "Encoder slots: EC1 right wheel, EC2 left wheel"
- note added: "IMU: LSM6DSV on the shared SPI bus"
- note added: "Motor current: TSC2020, 20 V/V across the 40 mOhm shunts"
- note added: "Sheet ports"
- note added: "Wall sensor 0: W1, emitter switch Q2"
- note added: "Wall sensor 1: W2, emitter switch Q3"
- note added: "Wall sensor 2: W3, emitter switch Q4"
- note added: "Wall sensor 3: W4, emitter switch Q5"
- title: (none) -> IMU, current sensors, wall sensors and encoder slots
- moved on the sheet: C24, C25, C26, C27, C28, C29, C67, C68, C69, C70, C71, C72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

Commit message: 🎨 Draw the diodes and buzzer as symbols, and make D4 blue
- 1N4148WS, B5819W and FUET-5030: replace the box bodies with diode,
  Schottky and buzzer symbols (same pins). Nudge D3 and BZ1 on both boards'
  PERIPHERALS sheets.
- D4: KENTO KT-0603B blue (C2288, VF 2.6-3.1 V at 5 mA) instead of the
  yellow NCD0603Y2. R4 goes from 680 Ohm to 100 Ohm: 1.2 mA at the worst
  bin and rail, 7.5 mA at most. LED_YELLOW_A is renamed LED_BLUE_A.
Changed lines of the file:
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@@
 		(dnp no)
 		(property "Reference" "D12"
-			(at 64.77 256.54 90)
+			(at 66.04 256.54 90)
 			(show_name no)
 			(do_not_autoplace no)
@@
 		)
 		(property "Value" "1N4148WS"
-			(at 64.77 259.08 90)
+			(at 66.04 259.08 90)
 			(show_name no)
 			(do_not_autoplace no)
@@
 		(dnp no)
 		(property "Reference" "D11"
-			(at 64.77 190.5 90)
+			(at 66.04 190.5 90)
 			(show_name no)
 			(do_not_autoplace no)
@@
 		)
 		(property "Value" "1N4148WS"
-			(at 64.77 193.04 90)
+			(at 66.04 193.04 90)
 			(show_name no)
 			(do_not_autoplace no)
@@
 		(dnp no)
 		(property "Reference" "D9"
-			(at 64.77 58.42 90)
+			(at 66.04 58.42 90)
 			(show_name no)
 			(do_not_autoplace no)
@@
 		)
 		(property "Value" "1N4148WS"
-			(at 64.77 60.96 90)
+			(at 66.04 60.96 90)
 			(show_name no)
 			(do_not_autoplace no)
@@
 		(dnp no)
 		(property "Reference" "D10"
-			(at 64.77 124.46 90)
+			(at 66.04 124.46 90)
 			(show_name no)
 			(do_not_autoplace no)
@@
 		)
 		(property "Value" "1N4148WS"
-			(at 64.77 127 90)
+			(at 66.04 127 90)
 			(show_name no)
 			(do_not_autoplace no)
@@
 	(wire
 		(pts
-			(xy 68.58 52.07) (xy 68.58 49.53)
+			(xy 68.58 55.88) (xy 68.58 49.53)
 		)
 		(stroke
@@
 	(wire
 		(pts
-			(xy 68.58 118.11) (xy 68.58 115.57)
+			(xy 68.58 121.92) (xy 68.58 115.57)
 		)
 		(stroke
@@
 	(wire
 		(pts
-			(xy 68.58 184.15) (xy 68.58 181.61)
+			(xy 68.58 187.96) (xy 68.58 181.61)
 		)
 		(stroke
@@
 	(wire
 		(pts
-			(xy 68.58 250.19) (xy 68.58 247.65)
+			(xy 68.58 254) (xy 68.58 247.65)
 		)
 		(stroke
@@
 	(symbol
 		(lib_id "GND")
-		(at 68.58 133.35 0)
+		(at 68.58 129.54 0)
 		(unit 1)
 		(body_style 1)
@@
 		(dnp no)
 		(property "Reference" "#PWR5690cf35e3415ed797620ba768beaec1"
-			(at 68.58 133.35 0)
+			(at 68.58 129.54 0)
 			(hide yes)
 			(show_name no)
@@
 		)
 		(property "Value" "GND"
-			(at 68.58 137.16 0)
+			(at 68.58 133.35 0)
 			(show_name no)
 			(do_not_autoplace no)
@@
 		)
 		(property "Footprint" ""
-			(at 68.58 133.35 0)
+			(at 68.58 129.54 0)
 			(hide yes)
 			(show_name no)
@@
 		)
 		(property "Datasheet" ""
-			(at 68.58 133.35 0)
+			(at 68.58 129.54 0)
 			(hide yes)
 			(show_name no)
@@
 		)
 		(property "Description" "Power symbol creates a global label with name \"GND\" , ground"
-			(at 68.58 133.35 0)
+			(at 68.58 129.54 0)
 			(hide yes)
 			(show_name no)
@@
 		)
 		(property "ki_keywords" "global power"
-			(at 68.58 133.35 0)
+			(at 68.58 129.54 0)
 			(hide yes)
 			(show_name no)
@@
 	(symbol
 		(lib_id "GND")
-		(at 68.58 199.39 0)
+		(at 68.58 195.58 0)
 		(unit 1)
 		(body_style 1)
@@
 		(dnp no)
 		(property "Reference" "#PWR52c876f83ef45f5297161084d11ef4e2"
-			(at 68.58 199.39 0)
+			(at 68.58 195.58 0)
 			(hide yes)
 			(show_name no)
@@
 		)
 		(property "Value" "GND"
-			(at 68.58 203.2 0)
+			(at 68.58 199.39 0)
 			(show_name no)
 			(do_not_autoplace no)
@@
 		)
 		(property "Footprint" ""
-			(at 68.58 199.39 0)
+			(at 68.58 195.58 0)
 			(hide yes)
 			(show_name no)
@@
 		)
 		(property "Datasheet" ""
-			(at 68.58 199.39 0)
+			(at 68.58 195.58 0)
 			(hide yes)
 			(show_name no)
@@
 		)
 		(property "Description" "Power symbol creates a global label with name \"GND\" , ground"
-			(at 68.58 199.39 0)
+			(at 68.58 195.58 0)
 			(hide yes)
 			(show_name no)
@@
 		)
 		(property "ki_keywords" "global power"
-			(at 68.58 199.39 0)
+			(at 68.58 195.58 0)
 			(hide yes)
 			(show_name no)
@@
 	(symbol
 		(lib_id "GND")
-		(at 68.58 265.43 0)
+		(at 68.58 261.62 0)
 		(unit 1)
 		(body_style 1)
@@
 		(dnp no)
 		(property "Reference" "#PWRb2a6ca0f2c9e56eda6d97f39b2ad1105"
-			(at 68.58 265.43 0)
+			(at 68.58 261.62 0)
 			(hide yes)
 			(show_name no)
@@
 		)
 		(property "Value" "GND"
-			(at 68.58 269.24 0)
+			(at 68.58 265.43 0)
 			(show_name no)
 			(do_not_autoplace no)
@@
 		)
 		(property "Footprint" ""
-			(at 68.58 265.43 0)
+			(at 68.58 261.62 0)
 			(hide yes)
 			(show_name no)
@@
 		)
 		(property "Datasheet" ""
-			(at 68.58 265.43 0)
+			(at 68.58 261.62 0)
 			(hide yes)
 			(show_name no)
@@
 		)
 		(property "Description" "Power symbol creates a global label with name \"GND\" , ground"
-			(at 68.58 265.43 0)
+			(at 68.58 261.62 0)
 			(hide yes)
 			(show_name no)
@@
 		)
 		(property "ki_keywords" "global power"
-			(at 68.58 265.43 0)
+			(at 68.58 261.62 0)
 			(hide yes)
 			(show_name no)
@@
 	(symbol
 		(lib_id "GND")
-		(at 68.58 67.31 0)
+		(at 68.58 63.5 0)
 		(unit 1)
 		(body_style 1)
@@
 		(dnp no)
 		(property "Reference" "#PWR78e36b8fa888579498bb26620b42abb1"
-			(at 68.58 67.31 0)
+			(at 68.58 63.5 0)
 			(hide yes)
 			(show_name no)
@@
 		)
 		(property "Value" "GND"
-			(at 68.58 71.12 0)
+			(at 68.58 67.31 0)
 			(show_name no)
 			(do_not_autoplace no)
@@
 		)
 		(property "Footprint" ""
-			(at 68.58 67.31 0)
+			(at 68.58 63.5 0)
 			(hide yes)
 			(show_name no)
@@
 		)
 		(property "Datasheet" ""
-			(at 68.58 67.31 0)
+			(at 68.58 63.5 0)
 			(hide yes)
 			(show_name no)
@@
 		)
 		(property "Description" "Power symbol creates a global label with name \"GND\" , ground"
-			(at 68.58 67.31 0)
+			(at 68.58 63.5 0)
 			(hide yes)
 			(show_name no)
@@
 		)
 		(property "ki_keywords" "global power"
-			(at 68.58 67.31 0)
+			(at 68.58 63.5 0)
 			(hide yes)
 			(show_name no)
