File: boards/main2/layout/main2.kicad_pcb (KiCad board)
At the start: 4 copper layers, 50 x 100 mm, 206 parts, among them IC1 STM32H725RGV6, IC2 LSM6DSVTR, IC6 STSPIN958TR, IC7 L6981C33DR, IC8 DRV8874PWPR, IC9 DRV8874PWPR, J1 B02B-PASK(LF)(SN), M1 B02B-PASK(LF)(SN), M2 B02B-PASK(LF)(SN), M3 B02B-PASK(LF)(SN), Q1 AO3400A, Q2 AO3400A, Q3 AO3400A, Q4 AO3400A, Q5 AO3400A, Q6 HSBB3072, Q8 AO3401A, Q9 AO3400A, SW1 DSHP04TJGER, SW2 GT-TC048B-H025-L1, SW3 GT-TC048B-H025-L1, SW4 SK-12D29-G060, U10 INA241A2IDGKR, U11 INA241A2IDGKR, U12 TLV9001IDBVR, U13 ESP32-S3-MINI-1-N8, U2 GT-USB-7010ASV, U6 USBLC6-2SC6, U8 ADP7142ACPZN3.3-R7

Commit message: 🎨 Draw the diodes and buzzer as symbols, and make D4 blue
- 1N4148WS, B5819W and FUET-5030: replace the box bodies with diode,
  Schottky and buzzer symbols (same pins). Nudge D3 and BZ1 on both boards'
  PERIPHERALS sheets.
- D4: KENTO KT-0603B blue (C2288, VF 2.6-3.1 V at 5 mA) instead of the
  yellow NCD0603Y2. R4 goes from 680 Ohm to 100 Ohm: 1.2 mA at the worst
  bin and rail, 7.5 mA at most. LED_YELLOW_A is renamed LED_BLUE_A.
Parts:
- D4: value LED YELLOW -> LED BLUE
- R4: value 680 1% -> 100 1%
Connections:
- net PERIPHERALS.LED_YELLOW_A renamed PERIPHERALS.LED_BLUE_A
