File: boards/main2/layout/REGULATORS.kicad_sch (KiCad schematic)
At the start: 30 parts, among them IC7 L6981C33DR, J1 B02B-PASK(LF)(SN), Q6 HSBB3072, Q8 AO3401A, SW4 SK-12D29-G060, U8 ADP7142ACPZN3.3-R7

Commit message: 🎨 Draw the diodes and buzzer as symbols, and make D4 blue
- 1N4148WS, B5819W and FUET-5030: replace the box bodies with diode,
  Schottky and buzzer symbols (same pins). Nudge D3 and BZ1 on both boards'
  PERIPHERALS sheets.
- D4: KENTO KT-0603B blue (C2288, VF 2.6-3.1 V at 5 mA) instead of the
  yellow NCD0603Y2. R4 goes from 680 Ohm to 100 Ohm: 1.2 mA at the worst
  bin and rail, 7.5 mA at most. LED_YELLOW_A is renamed LED_BLUE_A.
Changed lines of the file:
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@@
 		(dnp no)
 		(property "Reference" "D14"
-			(at 114.3 112.395 0)
+			(at 114.6175 113.665 0)
 			(show_name no)
 			(do_not_autoplace no)
@@
 		)
 		(property "Value" "B5819W"
-			(at 114.3 114.935 0)
+			(at 114.6175 116.205 0)
 			(show_name no)
 			(do_not_autoplace no)
@@
 	(wire
 		(pts
-			(xy 106.68 119.38) (xy 101.6 119.38)
+			(xy 110.49 119.38) (xy 101.6 119.38)
 		)
 		(stroke
@@
 	(wire
 		(pts
-			(xy 121.92 119.38) (xy 139.7 119.38)
-		)
-		(stroke
+			(xy 118.11 119.38) (xy 139.7 119.38)
+		)
+		(stroke

Commit message: 🚧 Swap main2's USB and ESP32-S3 for an ESP32-C5 and programming headers
Schematic and component checkpoint; the layout follows in its own commit.

- Remove USB-C, its ESD, power path and VBUS sense; both MCUs flash over
  the air.
- U13 ESP32-C5-MINI-1-N4 (dual-band, 5 GHz channels 36-48) in the
  rear-right corner, with its antenna notch on the right edge. SW4 and its
  notch move to the rear-left.
- H7-C5 link: SPI2 half-duplex 3-wire (PA12 SCK, PA11 CSn, PB14 DATA with
  IOSWP), PA9 flow control, UART4 fallback on the same pins. Fan_Enable
  moves to PB10, IMU INT1 to PB6, INT2 is left open.
- J2: 2x3 1.27 mm header in the ESP-Prog layout. SWD1: 1x4 1.27 mm in
  clone ST-Link order (SWDIO, GND, SWCLK, 5V). 5V_IN feeds VSYS through
  D17 (B5819W) to flash without the battery.
- R44/R45 to 20k/2k keeps PC5 below its absolute maximum at the clamp.
Parts:
- removed C63: 1uF 10% 25V X5R, stdlib_kicad-footprints_Capacitor_SMD:C_0402_1005Metric, symbol C_Small
- removed D16: 10V zener, Team-Micras_MicrasPCB_components_diodes_BZT52C10S:D_SOD-323, symbol BZT52C10S-7-F
- removed Q8: AO3401A, Team-Micras_MicrasPCB_components_aos_AO3401A:SOT-23, symbol AO3401A
- removed R56: 10k 1%, stdlib_kicad-footprints_Resistor_SMD:R_0402_1005Metric, symbol R_Small
- removed R57: 1M 1%, stdlib_kicad-footprints_Resistor_SMD:R_0402_1005Metric, symbol R_Small
- added D17: B5819W, Team-Micras_MicrasPCB_components_cj_B5819W:D_SOD-123, symbol B5819W
- R44: value 10k 1% -> 20k 1%
Connections:
- net VSYS: now also D17.1 (K)
- new net 5V_IN: D17.2 (A)
Other:
- note added: "VSYS: VBAT through D14, 5V_IN (a programmer's 5 V) through D17"
- note removed: "Power path: VSYS = VBAT or VBUS"
- title: Battery input, power path and regulators -> Battery input, VSYS and regulators
